File: kicad/outputs.kicad_sch (KiCad schematic)
At the start: 35 parts, among them J2 Thonkiconn, U4 TL074

Commit message: make 4hp
Parts:
- LED1, LED2, LED3, LED4: footprint Eurorack:LED 3mm -> allensynthesis:led-3mm
Changed lines of the file:
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@@
       (effects (font (size 1.27 1.27)) (justify right))
     )
-    (property "Footprint" "Eurorack:LED 3mm" (at 217.17 123.19 0)
+    (property "Footprint" "allensynthesis:led-3mm" (at 217.17 123.19 0)
       (effects (font (size 1.27 1.27)) hide)
     )
@@
       (effects (font (size 1.27 1.27)) (justify right))
     )
-    (property "Footprint" "Eurorack:LED 3mm" (at 97.79 123.19 0)
+    (property "Footprint" "allensynthesis:led-3mm" (at 97.79 123.19 0)
       (effects (font (size 1.27 1.27)) hide)
     )
@@
       (effects (font (size 1.27 1.27)) (justify right))
     )
-    (property "Footprint" "Eurorack:LED 3mm" (at 97.79 59.69 0)
+    (property "Footprint" "allensynthesis:led-3mm" (at 97.79 59.69 0)
       (effects (font (size 1.27 1.27)) hide)
     )
@@
       (effects (font (size 1.27 1.27)) (justify right))
     )
-    (property "Footprint" "Eurorack:LED 3mm" (at 217.17 59.69 0)
-      (effects (font (size 1.27 1.27)) hide)
-    )
+    (property "Footprint" "allensynthesis:led-3mm" (at 217.17 59.69 0)
+      (effects (font (size 1.27 1.27)) hide)
+    )

Commit message: reroute pcb
Parts:
- J2: footprint Eurorack:Thonkiconn Mono Jack -> allen-synthesis:jack-thonkiconn-mono
- LED1, LED2, LED3, LED4: footprint allensynthesis:led-3mm -> allen-synthesis:led-3mm
Changed lines of the file:
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@@
       (effects (font (size 1.27 1.27)) (justify right))
     )
-    (property "Footprint" "allensynthesis:led-3mm" (at 217.17 123.19 0)
+    (property "Footprint" "allen-synthesis:led-3mm" (at 217.17 123.19 0)
       (effects (font (size 1.27 1.27)) hide)
     )
@@
       (effects (font (size 1.27 1.27)) (justify right))
     )
-    (property "Footprint" "allensynthesis:led-3mm" (at 97.79 123.19 0)
+    (property "Footprint" "allen-synthesis:led-3mm" (at 97.79 123.19 0)
       (effects (font (size 1.27 1.27)) hide)
     )
@@
       (effects (font (size 1.27 1.27)) (justify right))
     )
-    (property "Footprint" "Eurorack:Thonkiconn Mono Jack" (at 241.3 41.91 0)
+    (property "Footprint" "allen-synthesis:jack-thonkiconn-mono" (at 241.3 41.91 0)
       (effects (font (size 1.27 1.27)) hide)
     )
@@
       (effects (font (size 1.27 1.27)) (justify right))
     )
-    (property "Footprint" "Eurorack:Thonkiconn Mono Jack" (at 241.3 105.41 0)
+    (property "Footprint" "allen-synthesis:jack-thonkiconn-mono" (at 241.3 105.41 0)
       (effects (font (size 1.27 1.27)) hide)
     )
@@
       (effects (font (size 1.27 1.27)) (justify right))
     )
-    (property "Footprint" "Eurorack:Thonkiconn Mono Jack" (at 121.92 41.91 0)
+    (property "Footprint" "allen-synthesis:jack-thonkiconn-mono" (at 121.92 41.91 0)
       (effects (font (size 1.27 1.27)) hide)
     )
@@
       (effects (font (size 1.27 1.27)) (justify right))
     )
-    (property "Footprint" "Eurorack:Thonkiconn Mono Jack" (at 121.92 105.41 0)
+    (property "Footprint" "allen-synthesis:jack-thonkiconn-mono" (at 121.92 105.41 0)
       (effects (font (size 1.27 1.27)) hide)
     )
@@
       (effects (font (size 1.27 1.27)) (justify right))
     )
-    (property "Footprint" "allensynthesis:led-3mm" (at 97.79 59.69 0)
+    (property "Footprint" "allen-synthesis:led-3mm" (at 97.79 59.69 0)
       (effects (font (size 1.27 1.27)) hide)
     )
@@
       (effects (font (size 1.27 1.27)) (justify right))
     )
-    (property "Footprint" "allensynthesis:led-3mm" (at 217.17 59.69 0)
-      (effects (font (size 1.27 1.27)) hide)
-    )
+    (property "Footprint" "allen-synthesis:led-3mm" (at 217.17 59.69 0)
+      (effects (font (size 1.27 1.27)) hide)
+    )

Commit message: add schematic notes
Connections:
- net at J2.3 (T), R9.1: no longer R6.2 (x4)
- net at R7.2, R9.2, U4.7: now also R6.2
- net at R7.2, R9.2, U4.14: now also R6.2
- net at R7.2, R9.2, U4.8: now also R6.2
- net at R7.2, R9.2, U4.1: now also R6.2
Other:
- note added: "A 1k resistor is in series with the final output to prevent the jack from shorting the op-amp output to ground when plugged half way in"
- note added: "The input is first RC low pass filtered to convert the PWM signal into a smooth DC voltage. The cutoff is approximately 1.6kHz"
- note added: "The output LED is tied directly to the output using a 5.6k resistor to prevent it from interfering with the signal itself"
- note added: "The signal is then amplified by ~3.3x for a range of ~0-10V There is a small amount of headroom so that the full 10V can be achieved even with low tolerance components"
- moved on the sheet: C13, C7, J2, LED1, LED2, LED3, LED4, R6, R7, R9, U4A, U4B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
