File: kicad/power.kicad_sch (KiCad schematic)
At the start: 6 parts, among them J2 Conn_02x08_Odd_Even

Commit message: make 4hp
Parts:
- removed D1: D, Diode_SMD:D_SOD-123, symbol Device:D
- removed J2: Conn_02x08_Odd_Even, Eurorack:Eurorack Power Header 16 Pin Unlabeled, symbol Connector_Generic:Conn_02x08_Odd_Even
- added C7 (x2): 100n, Capacitor_SMD:C_0402_1005Metric, symbol Device:C
- added J1: Conn_02x05_Odd_Even, Eurorack:Eurorack Power Header Unlabeled, symbol Connector_Generic:Conn_02x05_Odd_Even
- added U3: ~, Package_TO_SOT_SMD:SOT-89-3, symbol Eurorack:78L05G-AB3-R_5V_Linear_Voltage_Regulator_(JLC)
Connections:
- net +12V: now also C7.1, U3.3 (IN)
- net Earth: now also C7.2, C7.2, J1.3 (Pin_3), J1.4 (Pin_4), J1.5 (Pin_5), J1.6 (Pin_6), J1.7 (Pin_7), J1.8 (Pin_8), U3.2 (GND)
- net at D1.1 (K): now also J1.1 (Pin_1), J1.2 (Pin_2)
- net at D1.2 (A): now also J1.10 (Pin_10), J1.9 (Pin_9)
- new net +5V: C7.1, U3.1 (OUT)
Other:
- moved on the sheet: C25, C26, D1

Commit message: reroute pcb
Parts:
- J1: footprint Eurorack:Eurorack Power Header Unlabeled -> allen-synthesis:power-header-10-pin-unlabelled
Changed lines of the file:
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@@
       (effects (font (size 1.27 1.27)))
     )
-    (property "Footprint" "Eurorack:Eurorack Power Header Unlabeled" (at 39.37 41.91 0)
+    (property "Footprint" "allen-synthesis:power-header-10-pin-unlabelled" (at 39.37 41.91 0)
       (effects (font (size 1.27 1.27)) hide)
     )

Commit message: add schematic notes
Other:
- note added: "An internal +5V regulator is used to generate the supply for the XIAO RP2040 as using the 5V rail would require a 16 pin power header which would increase the width of the module"
- note added: "The series diodes protect the circuit by blocking any voltage with incorrect polarity which could occur if the power header was connected wrong"
- moved on the sheet: C25, C26, C7, D1, J1, U3
